File: bicolour-matrix/bicolour-matrix.kicad_sch (KiCad schematic)
At the start: 2 parts, among them J1 Conn_01x04_Pin

Commit message: feat: final revs
Parts:
- added C6: 10uF, PCM_JLCPCB:C_0805, symbol PCM_JLCPCB-Capacitors:0805,10uF
- added J2: Conn_01x04_Pin, Connector_PinHeader_2.54mm:PinHeader_1x04_P2.54mm_Vertical, symbol Connector:Conn_01x04_Pin
Connections:
- net GND: now also C6.2, J2.3 (Pin_3)
- net Matrix 1/SCL: now also J2.2 (Pin_2)
- net Matrix 1/SDA: now also J2.1 (Pin_1)
- net VDD: now also C6.1, J2.4 (Pin_4)
