File: bicolour-matrix/bicolour-matrix.kicad_pcb (KiCad board)
At the start: 2 copper layers, 136.8 x 33.5 mm, 52 parts, among them J1 Conn_01x04_Pin, J2 Conn_01x04_Pin, U1 HT16K33A-28SOP, U2 HT16K33A-28SOP, U3 HT16K33A-28SOP, U4 HT16K33A-28SOP

Commit message: feat: fixed lcsc component
Parts:
- U1, U2, U3, U4: value HT16K33A-28SOP -> HT16K33A-28SSOP
Changed lines of the file:
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@@
 			)
 		)
-		(property "Value" "HT16K33A-28SOP"
+		(property "Value" "HT16K33A-28SSOP"
 			(at -0.1 6.2 90)
 			(layer "F.Fab")
@@
 			)
 		)
-		(property "LCSC Part" "C5444737"
+		(property "LCSC Part" "C5444738"
 			(at 0 0 90)
 			(unlocked yes)
@@
 			)
 		)
-		(property "Value" "HT16K33A-28SOP"
+		(property "Value" "HT16K33A-28SSOP"
 			(at -0.1 6.2 90)
 			(layer "F.Fab")
@@
 			)
 		)
-		(property "LCSC Part" "C5444737"
+		(property "LCSC Part" "C5444738"
 			(at 0 0 90)
 			(unlocked yes)
@@
 			)
 		)
-		(property "Value" "HT16K33A-28SOP"
+		(property "Value" "HT16K33A-28SSOP"
 			(at -0.1 6.2 90)
 			(layer "F.Fab")
@@
 			)
 		)
-		(property "LCSC Part" "C5444737"
+		(property "LCSC Part" "C5444738"
 			(at 0 0 90)
 			(unlocked yes)
@@
 			)
 		)
-		(property "Value" "HT16K33A-28SOP"
+		(property "Value" "HT16K33A-28SSOP"
 			(at -0.1 6.2 90)
 			(layer "F.Fab")
@@
 			)
 		)
-		(property "LCSC Part" "C5444737"
+		(property "LCSC Part" "C5444738"
 			(at 0 0 90)
 			(unlocked yes)
