File: bicolour-matrix/matrix_module.kicad_sch (KiCad schematic)
At the start: 12 parts, among them U1 HT16K33A-28SOP

Commit message: feat: fixed lcsc component
Parts:
- U1: value HT16K33A-28SOP -> HT16K33A-28SSOP; LCSC Part C5444737 -> C5444738
Changed lines of the file:
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@@
 			)
 		)
-		(property "Value" "HT16K33A-28SOP"
+		(property "Value" "HT16K33A-28SSOP"
 			(at 121.9201 167.64 90)
 			(effects
@@
 			)
 		)
-		(property "LCSC Part" "C5444737"
+		(property "LCSC Part" "C5444738"
 			(at 123.19 120.65 0)
 			(effects
