File: adapter-board/adapter-board.kicad_pcb (KiCad board)
At the start: 2 copper layers, 136.8 x 33.5 mm, 9 parts, among them J1 Conn_01x02_Socket, J2 Conn_01x03_Pin, J3 Conn_01x01_Socket, J4 Conn_01x04_Socket, J5 Conn_01x04_Socket, U1 XIAO ESP32C3

Commit message: feat: gerbers
Routing:
- net GND: vias 59 -> 60
Changed lines of the file:
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@@
+	)
+	(via
+		(at 162.75 101.25)
+		(size 0.6)
+		(drill 0.3)
+		(layers "F.Cu" "B.Cu")
+		(free yes)
+		(net 4)
 	)
 	(via

Commit message: feat: final changes
Parts:
- J2: value Conn_01x03_Pin -> Conn_01x05_Pin; footprint Connector_PinHeader_2.54mm:PinHeader_1x03_P2.54mm_Horizontal -> Connector_PinHeader_2.54mm:PinHeader_1x05_P2.54mm_Horizontal; moved to B.Cu
- moved J2 7.68 mm to (153.4, 101.5)
Connections:
- J2 pad 3: GND -> Net-(J2-Pin_3)
- U1 pad 3: unconnected-(U1-D2-Pad3) -> Net-(J2-Pin_3)
- U1 pad 4: unconnected-(U1-D3-Pad4) -> Net-(J2-Pin_4)
Routing:
- net Net-(J2-Pin_4): track 0.00 -> 42.8 mm, vias 0 -> 2
- net Net-(J2-Pin_3): track 0.00 -> 29.0 mm, vias 0 -> 2
- net Net-(J2-Pin_1): track 25.1 -> 21.9 mm
- net VUSB: track 168.8 -> 167.3 mm
- net Net-(J2-Pin_2): track 25.9 -> 26.6 mm
- net GND: vias 60 -> 65

Commit message: feat: PCB updates
Parts:
- removed J3: Conn_01x01_Socket, custom:PinMatrix05x10P2.54
- added RZ1: RP2040-Zero, custom:RP2040-Zero, F.Cu at (182.8, 121.2)
- U1: value XIAO ESP32C3 -> ~; footprint xiao_esp32c3:xiao_esp32c3 -> custom:Generic-Level-Shifter
- moved U1 27.8 mm to (196.8, 113.8), turned to 0 degrees
- moved J1 5.60 mm to (112.5, 96.5)
- moved BT1 1.25 mm to (96.5, 102.0)
- moved U2 0.76 mm to (118.7, 96.2)
- moved J2 0.11 mm to (153.5, 101.4)
Connections:
- U1 pad 1: Net-(J2-Pin_1) -> Net-(J4-Pin_2)
- U1 pad 10: unconnected-(U1-D9-Pad10) -> GND
- U1 pad 11: Net-(BZ1-+) -> unconnected-(U1-LV3-Pad11)
- U1 pad 12: Net-(U1-VCC_3V3) -> unconnected-(U1-LV4-Pad12)
- U1 pad 2: Net-(J2-Pin_2) -> Net-(J4-Pin_1)
- U1 pad 3: Net-(J2-Pin_3) -> VUSB
- U1 pad 4: Net-(J2-Pin_4) -> GND
- U1 pad 5: Net-(J4-Pin_1) -> unconnected-(U1-HV3-Pad5)
- U1 pad 6: Net-(J4-Pin_2) -> unconnected-(U1-HV4-Pad6)
- U1 pad 7: unconnected-(U1-D6-Pad7) -> Net-(RZ1-GP5)
- U1 pad 8: unconnected-(U1-D7-Pad8) -> Net-(RZ1-GP4)
- U1 pad 9: unconnected-(U1-D8-Pad9) -> 3V3
- U2 pad 1: Net-(U1-VCC_3V3) -> VUSB
Routing:
- net Net-(U1-VCC_3V3): track 52.1 -> 0.00 mm, vias 1 -> 0
- net Net-(J4-Pin_2): track 206.3 -> 161.0 mm
- net Net-(RZ1-GP4): track 0.00 -> 39.0 mm
- net Net-(J4-Pin_1): track 206.9 -> 169.8 mm
- net 3V3: track 0.00 -> 33.9 mm
- net Net-(RZ1-GP5): track 0.00 -> 33.9 mm
- net VUSB: track 167.3 -> 197.4 mm, vias 1 -> 0
- net Net-(BZ1-+): track 56.1 -> 37.8 mm
- net Net-(J2-Pin_4): track 42.8 -> 25.2 mm, vias 2 -> 0
- net Net-(J2-Pin_1): track 21.9 -> 7.32 mm, vias 1 -> 0
- net Net-(J2-Pin_2): track 26.6 -> 13.9 mm, vias 1 -> 0
- net Net-(J2-Pin_3): track 29.0 -> 20.0 mm, vias 2 -> 0
- net unconnected-(BT1-+-Pad1): track 39.0 -> 42.8 mm, vias 0 -> 1
- net unconnected-(BT1---Pad2): track 19.3 -> 17.2 mm
- net GND: track 1.22 -> 0.00 mm, vias 65 -> 34
Other:
- outline, holes or cut-outs redrawn
- board text added: "GND"
