File: adapter-board/adapter-board.kicad_sch (KiCad schematic)
At the start: 0 parts

Commit message: feat: adapter board kicad
Parts:
- added BT1: Battery_Cell, Battery:BatteryHolder_Keystone_3034_1x20mm, symbol Device:Battery_Cell
- added BZ1: Buzzer, Buzzer_Beeper:Buzzer_12x9.5RM7.6, symbol Device:Buzzer
- added J1: Conn_01x02_Socket, Connector_PinHeader_2.54mm:PinHeader_1x02_P2.54mm_Vertical, symbol Connector:Conn_01x02_Socket
- added J2: Conn_01x03_Pin, Connector_PinHeader_2.54mm:PinHeader_1x03_P2.54mm_Horizontal, symbol Connector:Conn_01x03_Pin
- added J3: Conn_01x01_Socket, custom:PinMatrix05x10P2.54, symbol Connector:Conn_01x01_Socket
- added J4, J5: Conn_01x04_Socket, Connector_PinSocket_2.54mm:PinSocket_1x04_P2.54mm_Vertical, symbol Connector:Conn_01x04_Socket
- added U1: XIAO ESP32C3, xiao_esp32c3:xiao_esp32c3, symbol xiao_esp32c3:XIAO ESP32C3
- added U2: ~, Connector_PinHeader_2.54mm:PinHeader_1x05_P2.54mm_Vertical, symbol custom:DS3231-module
Connections:
- new net: BT1.1 (+), J1.1 (Pin_1)
- new net: BT1.2 (-), J1.2 (Pin_2)
- new net: J4.1 (Pin_1), J5.1 (Pin_1), U1.5 (D4), U2.2 (SDA)
- new net: J4.2 (Pin_2), J5.2 (Pin_2), U1.6 (D5), U2.3 (SCL)
- new net: U1.12 (VCC_3V3), U2.1 (VCC)
- new net: BZ1.1 (+), U1.11 (D10)
- new net: J2.1 (Pin_1), U1.1 (D0)
- new net: J2.2 (Pin_2), U1.2 (D1)
- new net GND: BZ1.2 (-), J2.3 (Pin_3), J4.3 (Pin_3), J5.3 (Pin_3), U1.13 (GND), U2.5 (GND)
- new net VUSB: J4.4 (Pin_4), J5.4 (Pin_4), U1.14 (VUSB)
- no-connect marks 0 -> 2
Other:
- note added: "DS3231 breakout board being used with B+ and B- pads that will be connected using wires manually"
- note added: "button board connector"

Commit message: feat: final changes
Parts:
- removed J2: Conn_01x03_Pin, Connector_PinHeader_2.54mm:PinHeader_1x03_P2.54mm_Horizontal, symbol Connector:Conn_01x03_Pin
- added J2: Conn_01x05_Pin, Connector_PinHeader_2.54mm:PinHeader_1x05_P2.54mm_Horizontal, symbol Connector:Conn_01x05_Pin
Connections:
- net GND: now also J2.5 (Pin_5)
- net at U1.1 (D0): now also J2.1 (Pin_1)
- net at U1.2 (D1): now also J2.2 (Pin_2)
- net at U1.3 (D2): now also J2.3 (Pin_3)
- net at U1.4 (D3): now also J2.4 (Pin_4)
Other:
- note added: "DS3231 Module"
Changed lines of the file:
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@@
 	(text "button board connector"
 		(exclude_from_sim no)
-		(at 67.564 26.924 0)
+		(at 54.864 17.018 0)
+		(effects
+			(font
+				(size 1.27 1.27)
+			)
+		)
+	)
+	(text "DS3231 Module"
+		(exclude_from_sim no)
+		(at 76.454 97.79 0)
 		(effects
 			(font
@@
 	(wire
 		(pts
+			(xy 50.8 44.45) (xy 55.88 44.45)
+		)
+		(stroke
+			(width 0)
+			(type default)
+		)
+	)
+	(wire
+		(pts
 			(xy 25.4 78.74) (xy 25.4 87.63)
 		)
@@
 	(wire
 		(pts
-			(xy 52.07 44.45) (xy 52.07 31.75)
+			(xy 53.34 40.64) (xy 55.88 40.64)
 		)
 		(stroke
@@
 	(wire
 		(pts
-			(xy 55.88 44.45) (xy 52.07 44.45)
-		)
-		(stroke
-			(width 0)
-			(type default)
-		)
-	)
-	(wire
-		(pts
 			(xy 96.52 52.07) (xy 91.44 52.07)
 		)
@@
 	(wire
 		(pts
+			(xy 53.34 34.29) (xy 53.34 40.64)
+		)
+		(stroke
+			(width 0)
+			(type default)
+		)
+	)
+	(wire
+		(pts
 			(xy 27.94 87.63) (xy 38.1 87.63)
 		)
@@
 	(wire
 		(pts
-			(xy 55.88 40.64) (xy 54.61 40.64)
-		)
-		(stroke
-			(width 0)
-			(type default)
-		)
-	)
-	(wire
-		(pts
 			(xy 27.94 55.88) (xy 52.07 55.88)
 		)
@@
 	(wire
 		(pts
+			(xy 48.26 48.26) (xy 55.88 48.26)
+		)
+		(stroke
+			(width 0)
+			(type default)
+		)
+	)
+	(wire
+		(pts
 			(xy 27.94 88.9) (xy 27.94 90.17)
 		)
@@
 	(wire
 		(pts
+			(xy 50.8 34.29) (xy 50.8 44.45)
+		)
+		(stroke
+			(width 0)
+			(type default)
+		)
+	)
+	(wire
+		(pts
 			(xy 91.44 78.74) (xy 81.28 78.74)
 		)
@@
 	(wire
 		(pts
-			(xy 54.61 31.75) (xy 54.61 40.64)
-		)
-		(stroke
-			(width 0)
-			(type default)
-		)
-	)
-	(wire
-		(pts
 			(xy 96.52 41.91) (xy 96.52 52.07)
 		)
@@
 	(wire
 		(pts
+			(xy 45.72 52.07) (xy 55.88 52.07)
+		)
+		(stroke
+			(width 0)
+			(type default)
+		)
+	)
+	(wire
+		(pts
+			(xy 45.72 34.29) (xy 45.72 52.07)
+		)
+		(stroke
+			(width 0)
+			(type default)
+		)
+	)
+	(wire
+		(pts
 			(xy 52.07 80.01) (xy 73.66 80.01)
 		)
@@
 		(pts
 			(xy 73.66 80.01) (xy 73.66 81.28)
+		)
+		(stroke
+			(width 0)
+			(type default)
+		)
+	)
+	(wire
+		(pts
+			(xy 48.26 34.29) (xy 48.26 48.26)
 		)
 		(stroke
@@
 	)
 	(symbol
+		(lib_id "power:GND")
+		(at 43.18 34.29 0)
+		(unit 1)
+		(exclude_from_sim no)
+		(in_bom yes)
+		(on_board yes)
+		(dnp no)
+		(fields_autoplaced yes)
+		(property "Reference" "#PWR01"
+			(at 43.18 40.64 0)
+			(effects
+				(font
+					(size 1.27 1.27)
+				)
+				(hide yes)
+			)
+		)
+		(property "Value" "GND"
+			(at 43.18 39.37 0)
+			(effects
+				(font
+					(size 1.27 1.27)
+				)
+			)
+		)
+		(property "Footprint" ""
+			(at 43.18 34.29 0)
+			(effects
+				(font
+					(size 1.27 1.27)
+				)
+				(hide yes)
+			)
+		)
+		(property "Datasheet" ""
+			(at 43.18 34.29 0)
+			(effects
+				(font
+					(size 1.27 1.27)
+				)
+				(hide yes)
+			)
+		)
+		(property "Description" "Power symbol creates a global label with name \"GND\" , ground"
+			(at 43.18 34.29 0)
+			(effects
+				(font
+					(size 1.27 1.27)
+				)
+				(hide yes)
+			)
+		)
+		(pin "1"
+		)
+		(instances
+			(project ""
+				(path "/49b15fa3-cd53-4d6b-9d74-1d88c955c2b1"
+					(reference "#PWR01")
+					(unit 1)
+				)
+			)
+		)
+	)
+	(symbol
 		(lib_id "Connector:Conn_01x02_Socket")
 		(at 107.95 87.63 0)
@@
 				(path "/49b15fa3-cd53-4d6b-9d74-1d88c955c2b1"
 					(reference "J4")
-					(unit 1)
-				)
-			)
-		)
-	)
-	(symbol
-		(lib_id "power:GND")
-		(at 49.53 31.75 0)
-		(unit 1)
-		(exclude_from_sim no)
-		(in_bom yes)
-		(on_board yes)
-		(dnp no)
-		(fields_autoplaced yes)
-		(property "Reference" "#PWR01"
-			(at 49.53 38.1 0)
-			(effects
-				(font
-					(size 1.27 1.27)
-				)
-				(hide yes)
-			)
-		)
-		(property "Value" "GND"
-			(at 49.53 36.83 0)
-			(effects
-				(font
-					(size 1.27 1.27)
-				)
-			)
-		)
-		(property "Footprint" ""
-			(at 49.53 31.75 0)
-			(effects
-				(font
-					(size 1.27 1.27)
-				)
-				(hide yes)
-			)
-		)
-		(property "Datasheet" ""
-			(at 49.53 31.75 0)
-			(effects
-				(font
-					(size 1.27 1.27)
-				)
-				(hide yes)
-			)
-		)
-		(property "Description" "Power symbol creates a global label with name \"GND\" , ground"
-			(at 49.53 31.75 0)
-			(effects
-				(font
-					(size 1.27 1.27)
-				)
-				(hide yes)
-			)
-		)
-		(pin "1"
-		)
-		(instances
-			(project ""
-				(path "/49b15fa3-cd53-4d6b-9d74-1d88c955c2b1"
-					(reference "#PWR01")
 					(unit 1)
 				)
@@
 	)
 	(symbol
-		(lib_id "Connector:Conn_01x03_Pin")
-		(at 52.07 26.67 270)
+		(lib_id "Connector:Conn_01x05_Pin")
+		(at 48.26 29.21 270)
 		(unit 1)
 		(exclude_from_sim no)
@@
 		(fields_autoplaced yes)
 		(property "Reference" "J2"
-			(at 52.07 21.59 90)
-			(effects
-				(font
-					(size 1.27 1.27)
-				)
-			)
-		)
-		(property "Value" "Conn_01x03_Pin"
-			(at 52.07 24.13 90)
-			(effects
-				(font
-					(size 1.27 1.27)
-				)
-			)
-		)
-		(property "Footprint" "Connector_PinHeader_2.54mm:PinHeader_1x03_P2.54mm_Horizontal"
-			(at 52.07 26.67 0)
+			(at 48.26 24.13 90)
+			(effects
+				(font
+					(size 1.27 1.27)
+				)
+			)
+		)
+		(property "Value" "Conn_01x05_Pin"
+			(at 48.26 26.67 90)
+			(effects
+				(font
+					(size 1.27 1.27)
+				)
+			)
+		)
+		(property "Footprint" "Connector_PinHeader_2.54mm:PinHeader_1x05_P2.54mm_Horizontal"
+			(at 48.26 29.21 0)
 			(effects
 				(font
@@
 		)
 		(property "Datasheet" "~"
-			(at 52.07 26.67 0)
-			(effects
-				(font
-					(size 1.27 1.27)
-				)
-				(hide yes)
-			)
-		)
-		(property "Description" "Generic connector, single row, 01x03, script generated"
-			(at 52.07 26.67 0)
-			(effects
-				(font
-					(size 1.27 1.27)
-				)
-				(hide yes)
-			)
+			(at 48.26 29.21 0)
+			(effects
+				(font
+					(size 1.27 1.27)
+				)
+				(hide yes)
+			)
+		)
+		(property "Description" "Generic connector, single row, 01x05, script generated"
+			(at 48.26 29.21 0)
+			(effects
+				(font
+					(size 1.27 1.27)
+				)
+				(hide yes)
+			)
+		)
+		(pin "5"
+		)
+		(pin "1"
 		)
 		(pin "2"
 		)
-		(pin "1"
-		)
 		(pin "3"
 		)
+		(pin "4"
+		)
 		(instances

Commit message: feat: PCB updates
Parts:
- removed J3: Conn_01x01_Socket, custom:PinMatrix05x10P2.54, symbol Connector:Conn_01x01_Socket
- removed U1: XIAO ESP32C3, xiao_esp32c3:xiao_esp32c3, symbol xiao_esp32c3:XIAO ESP32C3
- added RZ1: RP2040-Zero, custom:RP2040-Zero, symbol custom:RP2040-Zero
- added U1: ~, custom:Generic-Level-Shifter, symbol custom:Generic-Level-Shifter
Connections:
- net GND: now also RZ1.22 (GND), U1.10 (GND), U1.4 (GND)
- net VUSB: now also U2.1 (VCC), RZ1.23 (5V), U1.3 (HV)
- net at J4.1 (Pin_1), J5.1 (Pin_1), U2.2 (SDA): now also U1.2 (HV2)
- net at J4.2 (Pin_2), J5.2 (Pin_2), U2.3 (SCL): now also U1.1 (HV1)
- net at BZ1.1 (+): now also RZ1.11 (GP10)
- net at J2.1 (Pin_1): now also RZ1.1 (GP0)
- net at J2.2 (Pin_2): now also RZ1.2 (GP1)
- net at J2.3 (Pin_3): now also RZ1.3 (GP2)
- net at J2.4 (Pin_4): now also RZ1.4 (GP3)
- new net: RZ1.5 (GP4), U1.8 (LV2)
- new net: RZ1.6 (GP5), U1.7 (LV1)
- new net 3V3: RZ1.21 (3V3), U1.9 (LV)
Other:
- moved on the sheet: BT1, BZ1, J1, J2, J4, J5, U2
